File: PLC nizao/Circuitos Kicad/SDCARD y USB/PLC4UNI_MEZZANINE_PCB1.kicad_pcb (KiCad board)
At the start: 2 copper layers, 29.7 x 37.1 mm, 15 parts, among them J1 PZ254R-12-14P, U1 MC-121-L119

Commit message: Actualizando repositorio
Parts:
- added C3: 10uF, Capacitor_SMD_AKL:C_0603_1608Metric, F.Cu at (99.6, 94.5)
- added J2: FPC-05FB-30PH20, EasyEDA:FPC-SMD_30P-P0.50_FPC-05FB-30PH20, F.Cu at (108.5, 85.9)
- added R10: 6.8K, Resistor_SMD_AKL:R_0603_1608Metric, F.Cu at (102.4, 91.9)
- added R11: 300, Resistor_SMD_AKL:R_0603_1608Metric, F.Cu at (105.4, 94.2)
- added R12: 10K, Resistor_SMD_AKL:R_0603_1608Metric, F.Cu at (115.5, 91.9)
- added R13: 10K, Resistor_SMD_AKL:R_0603_1608Metric, F.Cu at (115.5, 94.7)
- added R14: 10K, Resistor_SMD_AKL:R_0603_1608Metric, F.Cu at (111.8, 91.7)
- added U2: MT9700-N, EasyEDA:SOT-23-5_L2.9-W1.6-P0.95-LS2.9-BL, F.Cu at (102.4, 94.5)
- J1: value PZ254R-12-14P -> PZ254R-12-16P; footprint EasyEDA:HDR-TH_14P-P2.54-H-M-R2-C7-S2.54 -> EasyEDA:HDR-TH_16P-P2.54-H-M-R2-C8-S2.54
- R3: value 10K -> 2.2K
- R4, R8: value 2.2K -> 10K
- moved R6 19.3 mm to (109.5, 94.2), turned to 90 degrees
- moved R7 16.0 mm to (107.4, 94.2), turned to 90 degrees
- moved L1 11.0 mm to (122.5, 81.6)
- moved R5 10.9 mm to (104.1, 81.8)
- moved R4 10.1 mm to (104.1, 79.1)
- moved R3 7.82 mm to (100.6, 81.5)
- moved R1 6.70 mm to (112.8, 81.3), turned to -90 degrees
- moved R2 6.68 mm to (101.6, 77.7), turned to -90 degrees
- moved R8 6.45 mm to (108.0, 79.4)
- moved R9 6.45 mm to (108.0, 82.1)
- moved C2 5.16 mm to (120.0, 84.1)
- moved J1 4.19 mm to (108.5, 98.6)
- moved C1 3.90 mm to (117.5, 81.6)
- moved Card1 1.54 mm to (118.6, 73.5)
- moved U1 1.45 mm to (103.4, 72.6)
Connections:
- net /clk renamed /SPI_CLK
- net /miso renamed /SPI_MISO
- net /mosi renamed /SPI_MOSI
- net /usb+ renamed /USB+
- net /usb- renamed /USB-
- Card1 pad 2: Net-(Card1-CD/DAT3) -> /SD_CS
- J1 pad 10: /i2c_scl -> /I2C_SCK
- J1 pad 11: /GPIO1 -> /RESET
- J1 pad 12: /GPIO2 -> /LCD_EN
- J1 pad 13: GND -> /LCD_CS
- J1 pad 14: GND -> /TP_INT
- J1 pad 3: /cs -> /SD_CS
- J1 pad 8: /i2c_sda -> /I2C_SDA
- R9 pad 2: Net-(Card1-CD/DAT3) -> /SD_CS
Other:
- board size 29.7 x 37.1 mm -> 30.2 x 37.7 mm
- board text added: "Design By Carlos Pichardo"
- board text added: "ITLA-HUB"
- board text added: "MAR 2026"
- board text added: "PLC4UNI MEZZANINE_PCB1"
