File: PLC nizao/Circuitos Kicad/SDCARD y USB/PLC4UNI_MEZZANINE_PCB1.kicad_sch (KiCad schematic)
At the start: 15 parts, among them J1 PZ254R-12-14P, U1 MC-121-L119

Commit message: Actualizando repositorio
Parts:
- removed J1: PZ254R-12-14P, EasyEDA:HDR-TH_14P-P2.54-H-M-R2-C7-S2.54, symbol EasyEDA:PZ254R-12-14P
- added C3: 10uF, Capacitor_SMD_AKL:C_0603_1608Metric, symbol Capacitor_AKL:C_0603
- added J1: PZ254R-12-16P, EasyEDA:HDR-TH_16P-P2.54-H-M-R2-C8-S2.54, symbol EasyEDA:PZ254R-12-16P
- added J2: FPC-05FB-30PH20, EasyEDA:FPC-SMD_30P-P0.50_FPC-05FB-30PH20, symbol EasyEDA:FPC-05FB-30PH20
- added R10: 6.8K, Resistor_SMD_AKL:R_0603_1608Metric, symbol Resistor_US_AKL:R_0603
- added R11: 300, Resistor_SMD_AKL:R_0603_1608Metric, symbol Resistor_US_AKL:R_0603
- added R12, R13, R14: 10K, Resistor_SMD_AKL:R_0603_1608Metric, symbol Resistor_US_AKL:R_0603
- added U2: MT9700-N, EasyEDA:SOT-23-5_L2.9-W1.6-P0.95-LS2.9-BL, symbol EasyEDA:MT9700-N
- R3: value 10K -> 2.2K
- R4, R8: value 2.2K -> 10K
Connections:
- net +3.3V: now also C3.1, J1.2, R12.1, R13.1, R14.1, U2.5 (VIN)
- net +5V: now also J1.1
- net GND: now also C3.2, J1.15, J1.16, J2.1, J2.21, J2.22, J2.23, J2.24, J2.30, J2.31, J2.32, R10.2, U2.2 (GND)
- net SD_CS: now reaches Card1.2 (CD/DAT3), R9.2
- net SD_CS: now also J1.3
- net clk renamed SPI_CLK
- net SPI_CLK: now also J1.9, J2.7
- net miso renamed SPI_MISO
- net SPI_MISO: now also J1.7, J2.8
- net mosi renamed SPI_MOSI
- net SPI_MOSI: now also J1.5, J2.10
- net usb+ renamed USB+
- net USB+: now also J1.4
- net usb- renamed USB-
- net USB-: now also J1.6
- new net: R10.1, U2.3 (SET)
- new net I2C_SCK: J1.10, J2.26
- new net I2C_SDA: J1.8, J2.27
- new net IM1: J2.4, R13.2
- new net IM2: J2.3, R12.2
- new net LCD_CS: J1.13, J2.6
- new net LCD_EN: J1.12, U2.4 (EN)
- new net LED+: J2.20, R11.2
- new net RD: J2.9
- new net RESET: J1.11, J2.29, J2.5, R14.2
- new net TP_INT: J1.14, J2.28
- new net VDD: J2.2, J2.25, R11.1, U2.1 (VOUT)
Other:
- moved on the sheet: C1, C2, Card1, L1, R1, R2, R3, R4, R5, R6, R7, R8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
